File: Hardware/Electrical/SCRAPPY_PCB/SCRAPPY_PCB.kicad_sch (KiCad schematic)
At the start: 54 parts, among them J1 Screw_Terminal_01x02, J2 Conn_01x04, J3 Conn_01x03, J4 Conn_01x03, J5 Conn_01x03, J6 Conn_01x04, J7 Conn_01x04, J8 Conn_01x04, J9 Conn_01x04, Q1 PN2222A, Q2 PN2222A, Q3 PN2222A, U1 ESP32-DevBoard, U2 L7805, U3 LM324

Commit message: Updated PCB; Ready for Manufacture
Parts:
- removed J7, J9: Conn_01x04, Connector_PinHeader_2.54mm:PinHeader_1x04_P2.54mm_Vertical, symbol Connector_Generic:Conn_01x04
- added D5: LED, LED_THT:LED_D5.0mm_Clear, symbol Device:LED
- added H1, H2, H3, H4: MountingHole, MountingHole:MountingHole_2.2mm_M2_DIN965_Pad, symbol Mechanical:MountingHole
- added J11: Conn_02x02_Odd_Even, Connector_PinHeader_2.54mm:PinHeader_1x04_P2.54mm_Vertical, symbol Connector_Generic:Conn_02x02_Odd_Even
- added J3: Conn_02x04_Counter_Clockwise, Connector_PinHeader_2.54mm:PinHeader_2x04_P2.54mm_Vertical, symbol Connector_Generic:Conn_02x04_Odd_Even
- added J6, J9: Conn_01x15, Connector_PinSocket_2.54mm:PinSocket_1x15_P2.54mm_Vertical, symbol Connector_Generic:Conn_01x15
- added R21: R, Resistor_THT:R_Axial_DIN0207_L6.3mm_D2.5mm_P10.16mm_Horizontal, symbol Device:R
- Q1, Q2, Q3: footprint Package_TO_SOT_THT:TO-92_Inline -> Package_TO_SOT_THT:TO-92_Inline_Wide
- U2: footprint Converter_DCDC:Converter_DCDC_Murata_OKI-78SR_Horizontal -> Converter_DCDC:Converter_DCDC_RECOM_R-78B-2.0_THT
- renumbered C4 to C1, C2 to C10, C6 to C2, C7 to C3, C9 to C4, C8 to C5, C10 to C6, C5 to C7, C3 to C8, C1 to C9, D4 to D1, D1 to D2, D2 to D4, J2 to J1, J3 to J10, J8 to J2, J1 to J4, J6 to J5, J4 to J7, J5 to J8, R14 to R1, R23 to R10, R21 to R11, R22 to R12, R11 to R13, R12 to R14, R9 to R15, R10 to R16, R8 to R17, R7 to R18, R6 to R19, R17 to R2, R5 to R20, R16 to R3, R18 to R4, R20 to R5, R13 to R6, R15 to R7, R19 to R8, R24 to R9, RV4 to RV2, RV2 to RV3, RV3 to RV4, U3 to U1, U1 to U3
Connections:
- net +12V: no longer C9.2
- net +3V3: now also J11.1 (Pin_1), J11.3 (Pin_3), J6.15 (Pin_15); no longer R16.1, R17.1, R19.1
- net +5V: now also C9.2, R16.1, R17.1, R19.1, J3.1 (Pin_1), J3.3 (Pin_3), J3.5 (Pin_5), J3.7 (Pin_7), J9.1 (Pin_1), J9.2 (Pin_2), R21.1; no longer R11.1
- net Aout_A: now also J9.15 (Pin_15)
- net Aout_B: now also J9.14 (Pin_14)
- net Aout_C: now also J9.12 (Pin_12)
- net Aout_D: now also J9.13 (Pin_13)
- net CS: now also J6.8 (Pin_8)
- net DC: now also U3.18 (*MTDO/GPIO15/ADC2_CH3), J6.13 (Pin_13); no longer U3.30 (GPIO23)
- net DIR_A: now also J6.9 (Pin_9)
- net DIR_B: now also U3.26 (GPIO21), J6.5 (Pin_5); no longer U3.13 (MTCK/GPIO13/ADC2_CH4)
- net DIR_C: now also J9.7 (Pin_7)
- net GND: now also D5.1 (K), J11.2 (Pin_2), J11.4 (Pin_4), J3.2 (Pin_2), J3.4 (Pin_4), J3.6 (Pin_6), J3.8 (Pin_8), J6.14 (Pin_14), J9.3 (Pin_3)
- net HALL-IN_A: now also U3.27 (U0RXD/GPIO3), J6.4 (Pin_4); no longer U3.26 (GPIO21)
- net HALL-IN_B: now also U3.28 (U0TXD/GPIO1), J6.3 (Pin_3); no longer U3.27 (U0RXD/GPIO3)
- net HALL-IN_C: now also J9.10 (Pin_10)
- net HALL-IN_D: now also J9.11 (Pin_11)
- net PCNT_A: now also J6.11 (Pin_11)
- net PCNT_B: now also U3.24 (GPIO18), J6.7 (Pin_7); no longer U3.11 (MTMS/GPIO14/ADC2_CH6)
- net PCNT_C: now also J9.9 (Pin_9)
- net PIN_1: now also J2.3 (Pin_3), U3.30 (GPIO23), J6.1 (Pin_1); no longer J2.1 (Pin_1), U3.18 (*MTDO/GPIO15/ADC2_CH3)
- net PIN_2: now also J6.12 (Pin_12)
- net PIN_3: now also J2.1 (Pin_1), U3.29 (GPIO22), J6.2 (Pin_2); no longer J2.3 (Pin_3), U3.28 (U0TXD/GPIO1)
- net PWM_A: now also J6.10 (Pin_10)
- net PWM_B: now also U3.25 (GPIO19), J6.6 (Pin_6); no longer U3.12 (*MTDI/GPIO12/ADC2_CH5)
- net PWM_C: now also J9.8 (Pin_8)
- net RES: now also U3.13 (MTCK/GPIO13/ADC2_CH4), J9.4 (Pin_4); no longer U3.29 (GPIO22)
- net SCLK: now also U3.11 (MTMS/GPIO14/ADC2_CH6), J9.6 (Pin_6); no longer U3.24 (GPIO18)
- net SDA: now also U3.12 (*MTDI/GPIO12/ADC2_CH5), J9.5 (Pin_5); no longer U3.25 (GPIO19)
- new net: D5.2 (A), R21.2
Other:
- moved on the sheet: C9, J2, U3
